File: KiCad/4S-Li-ion-battery-meter/4S-Li-ion-battery-meter.kicad_sch (KiCad schematic)
At the start: 25 parts, among them J1 Conn_01x02_Pin, SW1 SW_Push, U1 LM339

Commit message: Sent to production!
Parts:
- RV1: footprint Potentiometer_SMD:Potentiometer_Bourns_3214J_Horizontal -> Potentiometer_SMD:Potentiometer_Bourns_TC33X_Vertical
Changed lines of the file:
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@@
 			)
 		)
-		(property "Footprint" "Potentiometer_SMD:Potentiometer_Bourns_3214J_Horizontal"
+		(property "Footprint" "Potentiometer_SMD:Potentiometer_Bourns_TC33X_Vertical"
 			(at 88.9 118.11 0)
 			(effects
