File: KiCad/relay-hat-v2/relay-hat-v2.kicad_sch (KiCad schematic)
At the start: 21 parts, among them J1 Screw_Terminal_01x04, J10 Screw_Terminal_01x02, J2 Conn_01x04_Pin, J3 Screw_Terminal_01x02, J4 Screw_Terminal_01x02, J5 Screw_Terminal_01x02, J6 Screw_Terminal_01x02, J7 Screw_Terminal_01x02, J8 Screw_Terminal_01x02, J9 Screw_Terminal_01x02, U1 TCA9554PW, U10 TMP1075DGKR, U2 TPS2051CDBV, U3 TPS2051CDBV, U4 TPS2051CDBV, U5 TPS2051CDBV, U6 TPS2051CDBV, U7 TPS2051CDBV, U8 TPS2000CDGK, U9 TPS2000CDGK

Commit message: Updated some code and micro-some-brero
Parts:
- U8, U9: value TPS2000CDGK -> TPS2001CDGK
Changed lines of the file:
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@@
 			)
 		)
-		(property "Value" "TPS2000CDGK"
+		(property "Value" "TPS2001CDGK"
 			(at 173.99 93.98 0)
 			(effects
@@
 			)
 		)
-		(property "Value" "TPS2000CDGK"
+		(property "Value" "TPS2001CDGK"
 			(at 173.99 68.58 0)
 			(effects
